File: light_controller.brd (EAGLE design)
At the start: 100 x 80 mm, 96 parts, among them IC1 ULN2803A, U1 DAC5578SPW, U2 LM3480IM3-5.0, U3 RCD-24-0.70

Commit message: updated all elements in schematic to be from openag_eagle_library repo
Parts:
- removed C12: 4.7uF, rcl:C1206
- removed C13: 0.1uF, rcl:C0603
- removed F6: (no value), fuse:GSH15
- removed IC1: ULN2803A, uln-udn:DIL18
- removed LED9: (no value), led:SMARTLED-TTW
- removed R17: 10k, rcl:R0603
- removed R18, R19, R20, R21, R25, R26, R27, R28: 0 ohm, rcl:R0603
- removed R24: 10 ohm, rcl:R0603
- removed R29, R30: 1K, rcl:R0603
- removed RELAY_1: G5LE-14_DC12, relay_2:RELAY_G5LE-1
- removed S1: (no value), switch-omron:B3F-10XX
- removed U$2: PHOTON_WITH_HEADERS, Spark:PHOTON
- removed U$4: SMAJ14A, openag_diodes:DO-214AC
- added *CH7+, *CH7-: WIREPAD3,17/1,3, wirepad:3,17/1,3
- added C19, C20: 10uF, openag-capacitors:C1206
- added D1: SMAJ14A, openag-diodes:DO-214AC
- added F2, F3: SST 7, openag-fuses:SS
- added IC2: ULN2803A, openag-transistors:DIL18
- added LED2: (no value), openag-diodes:CHIPLED_0603
- added R10, R13, R14, R15, R8, R9: 0 ohm, openag-resistors:RC0603N
- added R3, R4: 10K, openag-resistors:RC0603N
- added R5, R6, R7: 1K, openag-resistors:RC0603N
- added TP26, TP27: PTR1B2,54, testpad:B2,54
- added U4: G5LE-14 DC24, openag-relays:RELAY_G5LE-1
- added U5: ISO1540DR, openag-isolators:D8
- C1: value 1uF -> 4.7uF; device rcl:C0603 -> openag-capacitors:CAP_C1206
- C10, C3, C5: device rcl:C1206 -> openag-capacitors:CAP_C1206
- C11, C8: value 10uF -> 0.1uF; device rcl:C1206 -> openag-capacitors:C1206C
- C2, C6: device rcl:C0603 -> openag-capacitors:C1206C
- C4: device rcl:C1206 -> openag-capacitors:C1206
- C7: value 10uF -> 1uF; device rcl:C1206 -> openag-capacitors:C1206
- C9: value 0.1uF -> 10uF; device rcl:C0603 -> openag-capacitors:C1206
- F1: value (none) -> SST 7; device fuse:GSH15 -> openag-fuses:SS
- LED1: device led:CHIP-LED0603 -> openag-diodes:CHIPLED_0603
- R1: value 10K -> 10 ohm; device rcl:R0603 -> openag-resistors:RC0603N
- R11, R12: value 1K -> 0 ohm; device rcl:R0603 -> openag-resistors:RC0603N
- R2: value 0 ohm -> 1K; device rcl:R0603 -> openag-resistors:RC0603N
- TP1, TP2: device testpad:B2,54 -> openag-testpoints:B2,54
- U$1: value PSOC_4000 -> PHOTON_WITH_HEADERS; device stovelite:SOIC16 -> openag-microcontrollers:PHOTON
- U$3: value ISO1540 -> PSOC_4000; device ISO1540:SOIC8 -> openag-microcontrollers:SOIC16
- U2: device LEDdynamics:SOT-23 -> openag-regulators:SOT-23
- moved C9 1673.0 mm to (-363.2, -1503.7)
- moved C10 1672.9 mm to (-361.9, -1510.0)
- moved R1 1537.2 mm to (-369.6, -1540.5)
- moved R2 1355.2 mm to (-306.1, -1397.0)
- moved TP1 1348.6 mm to (-255.3, -1333.5)
- moved TP2 1348.6 mm to (-255.3, -1339.8)
- moved F1 1335.6 mm to (-264.2, -1337.3)
- moved U2 1136.9 mm to (-372.1, -1516.4)
- moved U$1 1117.5 mm to (-350.5, -1461.8)
- moved C4 1116.9 mm to (-370.8, -1522.7)
- moved C6 1116.9 mm to (-369.6, -1535.4)
- moved C5 1116.6 mm to (-369.6, -1529.1)
- moved C3 1082.1 mm to (-354.3, -1470.7)
- moved C2 1068.9 mm to (-317.5, -1433.8)
- moved C1 1067.7 mm to (-317.5, -1427.5)
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Connections:
- removed net +12V: IC1.10, R24.1, RELAY_1.1, RELAY_1.2
- removed net 1C: IC1.18, RELAY_1.5, TP1.TP
- removed net N$13: LED9.A@1, R17.1
- removed net N$4: IC1.1, R2.2
- removed net P0: R17.2, R2.1
- removed net R1: F1.2, R1.2, TP2.TP
- new net CH7-: *CH7-.1, F1.2, R3.2, TP2.TP, TP27.TP
- new net DIM2: U1.13
- new net DIM3: U1.5
- new net DIM4: U1.12
- new net DIM5: U1.6
- new net DIM6: U1.11
- new net N$5: F3.1, U3.6
- new net N$7: LED2.A, R4.1
- new net O1: IC2.18, TP1.TP, U4.5
- new net P6: U$3.11
- new net P7: IC2.1, R4.2, U$3.10
- net +24V: now also *CH7+.1, F2.2, IC2.10, R1.1, TP26.TP, U4.1, U4.2; no longer F6.2
- net +3V3: now also C1.1, C20.1, R2.2, R5.2, R8.2, U$3.7, U5.8; no longer C3.1, C8.1, R18.2, R29.2, R30.2, S1.2, U$1.7, U$3.8
- net 24V_IN: now also C10.1, C9.1, D1.C, F2.1; no longer C12.1, C13.1, F6.1, U$4.C
- net CH1+: now also F3.2; no longer U3.6
- net GND1: now also C19.2, U5.4; no longer C7.2, U$3.4
- net GND2: now also C20.2, C7.2, D1.A, IC2.9, LED2.C, U$1.2, U$1.21, U$3.8, U5.5; no longer C12.2, C13.2, IC1.9, LED9.C@1, U$1.8, U$2.2, U$2.21, U$3.5, U$4.A
- net I2C_3V3: now also C19.1, R6.2, R7.2, U5.1; no longer C7.1, R11.2, R12.2, U$3.1
- net I2C_SCL: now also R6.1, R7.1, U5.3; no longer R12.1, U$3.3
- net I2C_SDA: now also U5.2; no longer R11.1, U$3.2
- net N$1: now also R3.1; no longer R1.1
- net N$2: now also U4.3; no longer RELAY_1.3
- net N$21: now also R13.1, U$1.15; no longer R26.1, U$2.15
- net N$22: now also R14.1, U$1.14; no longer R27.1, U$2.14
- net N$23: now also C3.1, C8.1, R8.1, U$1.24; no longer C10.1, C9.1, R18.1, U$2.24
- net N$24: now also R9.1, U$1.19; no longer R19.1, U$2.19
- net N$25: now also R10.1, U$1.18; no longer R20.1, U$2.18
- net N$26: now also R11.1, U$1.17; no longer R21.1, U$2.17
- net N$27: now also R12.1, U$1.16; no longer R25.1, U$2.16
- net N$28: now also R15.1, U$1.13; no longer R28.1, U$2.13
- net N$29: now also C7.1, U$3.6; no longer C1.1, U$1.6
- net N$39: now also R1.2; no longer R24.2
- net P1: now also R9.2, U$3.16; no longer R19.2, S1.4, U$1.16
- net P2: now also R10.2, U$3.15; no longer R20.2, U$1.15
- net P3: now also R11.2, U$3.14; no longer R21.2, U$1.14
- net P4: now also R12.2, U$3.13; no longer R25.2, U$1.13
- net P5: now also R13.2, U$3.12; no longer R26.2, U$1.12
- net SCL: now also R14.2, R5.1, U$3.2, U5.6; no longer R27.2, R30.1, U$1.2, U$3.6
- net SDA: now also R15.2, R2.1, U$3.1, U5.7; no longer R28.2, R29.1, U$1.1, U$3.7
- net VBAT: now also U$1.22; no longer U$2.22
- net VIN: now also U$1.1; no longer U$2.1

Commit message: calculated power consuption, cleaned up mcu 0ohnm resistors
Parts:
- removed *CH7+, *CH7-: WIREPAD3,17/1,3, wirepad:3,17/1,3
- removed C4: 10uF, openag-capacitors:C1206
- removed C5: 4.7uF, openag-capacitors:CAP_C1206
- removed C6: 0.1uF, openag-capacitors:C1206C
- removed F1: SST 7, openag-fuses:SS
- removed IC2: ULN2803A, openag-transistors:DIL18
- removed LED1, LED2: (no value), openag-diodes:CHIPLED_0603
- removed R1: 10 ohm, openag-resistors:RC0603N
- removed TP1, TP2: PTR1B2,54, openag-testpoints:B2,54
- removed TP11, TP26, TP27: PTR1B2,54, testpad:B2,54
- removed U2: LM3480IM3-5.0, openag-regulators:SOT-23
- removed U4: G5LE-14 DC24, openag-relays:RELAY_G5LE-1
- added R16, R17, R18, R20, R21, R22, R23, R24, R25, R26, R27, R28, R29, R30, R31, R32, R33: 0 ohm, openag-resistors:RC0603N
- C1: value 4.7uF -> 1uF; device openag-capacitors:CAP_C1206 -> openag-capacitors:C1206
- C7: value 1uF -> 0.1uF; device openag-capacitors:C1206 -> openag-capacitors:C1206C
- R3, R4: value 10K -> 0 ohm
- moved R3 271.9 mm to (-369.6, -1602.7)
- moved R4 245.0 mm to (-369.6, -1606.5)
- moved C1 149.5 mm to (-370.8, -1567.2)
- moved C7 148.6 mm to (-369.6, -1560.8)
Connections:
- removed net CH7-: *CH7-.1, F1.2, R3.2, TP2.TP, TP27.TP
- removed net N$39: C4.1, R1.2, U2.2
- removed net O1: IC2.18, TP1.TP, U4.5
- new net N$10: R21.1, U$3.15
- new net N$11: R22.1, U$3.14
- new net N$12: R23.1, U$3.13
- new net N$13: R24.1, U$3.12
- new net N$14: R25.1, U$3.11
- new net N$15: C7.2, R26.2
- new net N$16: C1.1, C2.1, R27.1, U$3.7
- new net N$17: C1.2, C2.2, R28.2
- new net N$18: R29.2, U$3.8
- new net N$19: R30.2, U$1.2
- new net N$20: C3.2, C8.2, R31.2
- new net N$30: R32.1, U$1.21
- new net N$31: R33.1, U$3.10
- new net N$4: R16.1, U$1.7
- new net N$6: R17.1, U$1.8
- new net N$8: R18.2, U1.9
- net +24V: no longer *CH7+.1, IC2.10, R1.1, TP26.TP, U4.1, U4.2
- net +3V3: now also R27.2; no longer C1.1, C2.1, C5.1, C6.1, TP11.TP, U$3.7, U2.3
- net GND2: now also R26.1, R28.1, R29.1, R30.1, R31.1, R32.2; no longer C1.2, C2.2, C3.2, C4.2, C5.2, C6.2, C7.2, C8.2, IC2.9, LED1.C, LED2.C, U$1.2, U$1.21, U$3.8, U2.1
- net N$1: now also R3.2, U$3.1; no longer LED1.A, R3.1
- net N$2: now also R4.2, U$3.2; no longer F1.1, U4.3
- net N$7: now also R20.1, U$3.16; no longer LED2.A, R4.1
- net P1: now also R20.2; no longer U$3.16
- net P2: now also R21.2; no longer U$3.15
- net P3: now also R22.2; no longer U$3.14
- net P4: now also R23.2; no longer U$3.13
- net P5: now also R24.2; no longer U$3.12
- net P6: now also R16.2, R25.2; no longer U$3.11
- net P7: now also R17.2, R18.1, R33.2; no longer IC2.1, R4.2, U$3.10
- net SCL: now also R4.1; no longer U$3.2
- net SDA: now also R3.1; no longer U$3.1

Commit message: added 3v3 syncronous regulator module
Parts:
- removed U$1: PHOTON_WITH_HEADERS, openag-microcontrollers:PHOTON
- removed U$3: PSOC_4000, openag-microcontrollers:SOIC16
- added C4: 22uF, openag-capacitors:C1206
- added C5: 10uF, openag-capacitors:C1206
- added R1: 100K, openag-resistors:RC0603N
- added R34: 51K, openag-resistors:RC0603N
- added R35: 160K, openag-resistors:RC0603N
- added U$2: CY8C4013SXI-41, openag-microcontrollers:SOIC16
- added U2: MPM3620GQV-P, openag-regulators:20-POWERLFQFN-MODULE
- added U4: PHOTONH, openag-microcontrollers:PHOTON
Connections:
- new net N$32: R1.1, U2.17
- new net N$33: R34.2, R35.1, U2.1
- net +24V: now also C5.1, R1.2, U2.16
- net +3V3: now also C4.1, R35.2, U2.7, U2.8, U2.9
- net GND2: now also C4.2, C5.2, R34.1, U2.3
- net N$1: now also U$2.1; no longer U$3.1
- net N$10: now also U$2.15; no longer U$3.15
- net N$11: now also U$2.14; no longer U$3.14
- net N$12: now also U$2.13; no longer U$3.13
- net N$13: now also U$2.12; no longer U$3.12
- net N$14: now also U$2.11; no longer U$3.11
- net N$16: now also U$2.7; no longer U$3.7
- net N$18: now also U$2.8; no longer U$3.8
- net N$19: now also U4.2; no longer U$1.2
- net N$2: now also U$2.2; no longer U$3.2
- net N$21: now also U4.15; no longer U$1.15
- net N$22: now also U4.14; no longer U$1.14
- net N$23: now also U4.24; no longer U$1.24
- net N$24: now also U4.19; no longer U$1.19
- net N$25: now also U4.18; no longer U$1.18
- net N$26: now also U4.17; no longer U$1.17
- net N$27: now also U4.16; no longer U$1.16
- net N$28: now also U4.13; no longer U$1.13
- net N$29: now also U$2.6; no longer U$3.6
- net N$30: now also U4.21; no longer U$1.21
- net N$31: now also U$2.10; no longer U$3.10
- net N$4: now also U4.7; no longer U$1.7
- net N$6: now also U4.8; no longer U$1.8
- net N$7: now also U$2.16; no longer U$3.16
- net VBAT: now also U4.22; no longer U$1.22
- net VIN: now also U4.1; no longer U$1.1

Commit message: added x2y cap for 24v conditioning and testpoints for self-contined module testing
Parts:
- removed R11, R12, R13, R16, R17, R20, R21, R22, R23, R24, R25, R33: 0 ohm, openag-resistors:RC0603N
- added CX1: 0.1uF, openag-capacitors:CX1206
- added TP1, TP11, TP2, TP26, TP27, TP28, TP29, TP30, TP31, TP32, TP33, TP34: PTR1B2,54, openag-testpoints:B2,54
- TP10, TP12, TP13, TP14, TP15, TP16, TP17, TP18, TP19, TP20, TP21, TP22, TP23, TP24, TP25, TP3, TP4, TP5, TP6, TP7, TP8, TP9: device testpad:B2,54 -> openag-testpoints:B2,54
- moved TP25 2398.0 mm to (-429.3, -1868.2)
- moved TP24 2390.7 mm to (-429.3, -1861.8)
- moved TP10 2276.1 mm to (-429.3, -1747.5)
- moved TP9 2268.8 mm to (-429.3, -1741.2)
- moved TP8 2261.5 mm to (-429.3, -1734.8)
- moved TP7 2231.5 mm to (-429.3, -1728.5)
- moved TP4 2193.1 mm to (-429.3, -1766.6)
- moved TP6 2151.0 mm to (-429.3, -1722.1)
- moved TP5 2143.6 mm to (-429.3, -1715.8)
- moved TP3 2116.3 mm to (-429.3, -1690.4)
- moved TP19 770.3 mm to (-429.3, -1849.1)
- moved TP15 764.3 mm to (-429.3, -1817.4)
- moved TP23 752.3 mm to (-429.3, -1855.5)
- moved TP21 746.3 mm to (-429.3, -1836.4)
- moved TP20 746.3 mm to (-429.3, -1830.1)
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Connections:
- removed net N$10: R21.1, U$2.15
- removed net N$11: R22.1, U$2.14
- removed net N$12: R23.1, U$2.13
- removed net N$13: R24.1, U$2.12
- removed net N$14: R25.1, U$2.11
- removed net N$21: R13.1, U4.15
- removed net N$24: R9.1, U4.19
- removed net N$25: R10.1, U4.18
- removed net N$26: R11.1, U4.17
- removed net N$27: R12.1, U4.16
- removed net N$31: R33.1, U$2.10
- removed net N$6: R17.1, U4.8
- removed net P2: R10.2, R21.2
- removed net P3: R11.2, R22.2
- removed net P4: R12.2, R23.2
- removed net P5: R13.2, R24.2
- removed net P6: R16.2, R25.2
- removed net P7: R17.2, R18.1, R33.2
- net +24V: now also TP1.TP, TP23.TP
- net +3V3: now also TP19.TP, TP3.TP, TP5.TP
- net 24V_IN: now also CX1.1, CX1.2; no longer TP21.TP
- net CH1+: no longer TP12.TP
- net CH1-: now also TP18.TP; no longer TP13.TP
- net CH2+: no longer TP14.TP
- net CH2-: no longer TP15.TP
- net CH3+: no longer TP16.TP
- net CH3-: no longer TP17.TP
- net CH4+: no longer TP7.TP
- net CH4-: no longer TP8.TP
- net CH5+: no longer TP9.TP
- net CH5-: no longer TP10.TP
- net CH6+: no longer TP24.TP
- net CH6-: no longer TP25.TP
- net DIM1: now also TP13.TP
- net GND1: now also TP12.TP; no longer TP20.TP, TP4.TP
- net GND2: now also CX1.3, CX1.4, TP14.TP, TP2.TP, TP20.TP, TP4.TP, TP8.TP; no longer TP18.TP
- net I2C_3V3: now also TP9.TP; no longer TP23.TP, TP6.TP
- net I2C_SCL: now also TP11.TP; no longer TP19.TP, TP3.TP
- net I2C_SDA: now also TP10.TP; no longer TP22.TP, TP5.TP
- net N$1: now also TP31.TP
- net N$16: now also TP34.TP
- net N$18: now also TP33.TP
- net N$19: now also TP24.TP
- net N$2: now also TP32.TP
- net N$22: now also TP27.TP
- net N$23: now also TP25.TP
- net N$28: now also TP28.TP
- net N$3: now also TP16.TP
- net N$30: now also TP26.TP
- net N$4: now also R9.1, TP30.TP, U$2.11; no longer R16.1, U4.7
- net N$5: now also TP17.TP
- net N$7: now also R10.1, TP29.TP, U4.15; no longer R20.1, U$2.16
- net N$8: now also TP15.TP
- net P1: now also R10.2, R18.1; no longer R20.2
- net SCL: now also TP21.TP, TP7.TP
- net SDA: now also TP22.TP, TP6.TP

Commit message: routed current regulators and 3.3v sync regulators, added rs485 to ttl transceiver
Parts:
- removed I2C_3V3_IN, I2C_3V3_OUT, I2C_GND_IN, I2C_GND_OUT, I2C_SCL_IN, I2C_SCL_OUT, I2C_SDA_IN, I2C_SDA_OUT: WIREPAD3,17/1,3, wirepad:3,17/1,3
- removed R26, R28, R29, R30: 0 ohm, openag-resistors:RC0603N
- removed TP10, TP11, TP12, TP15, TP19, TP20, TP21, TP22, TP23, TP24, TP25, TP26, TP27, TP28, TP29, TP30, TP31, TP32, TP33, TP34, TP4, TP9: PTR1B2,54, openag-testpoints:B2,54
- added 3V3_IN, 3V3_OUT, 5V_IN, 5V_OUT, GND_IN, GND_OUT, RX_IN, RX_OUT, SCL_IN, SCL_OUT, SDA_IN, SDA_OUT, TX_IN, TX_OUT, _GND_IN, _GND_OUT: (no value), openag-wirepads:3,17/1,3
- added C12, C21, C22, C24, C25, C27, C28, C30, C31, C6: 10uF, openag-capacitors:C1206
- added C13, C23, C26, C29, C32: 100uF, openag-capacitors:EEE-1HA101UP
- added C33: 330pF, openag-capacitors:C1206
- added F1, F4, F5, F6, F7: SST 7, openag-fuses:SS
- added L2, L3, L4, L5, L6: 120uH, openag-inductors:74404064121
- added R11: 6.34 ohm, openag-resistors:R0805
- added R12: 16.5K, openag-resistors:RC0603N
- added TP35, TP36, TP37, TP38, TP39, TP40, TP41, TP42, TP43, TP44, TP45, TP46, TP47, TP48, TP49, TP50, TP51, TP52, TP53, TP54, TP55, TP56, TP57, TP58, TP59: PTR1B2,54, openag-testpoints:B2,54
- added U10, U6, U7, U8, U9: RCD-24-0.70, openag-regulators:RCD-24-PINNED
- added U11: MAX3485CSA+T, openag-transceivers:SOIC8
- +24V, CH1+, CH1-, CH2+, CH2-, CH3+, CH3-, CH4+, CH4-, CH5+, CH5-, CH6+, CH6-, GND: value WIREPAD3,17/1,3 -> (none); device wirepad:3,17/1,3 -> openag-wirepads:3,17/1,3
- R1: value 100K -> 200K
- moved R9 1927.2 mm to (67.3, 78.7)
- moved R10 1920.2 mm to (29.2, 77.5)
- moved TP16 1910.4 mm to (14.0, 59.9)
- moved TP14 1889.8 mm to (5.08, 59.9)
- moved TP8 1889.7 mm to (61.0, 90.2)
- moved TP13 1884.8 mm to (10.2, 59.9)
- moved TP7 1881.6 mm to (53.3, 90.2)
- moved TP18 1880.9 mm to (5.08, 19.1)
- moved TP17 1876.5 mm to (12.7, 19.1)
- moved TP6 1874.5 mm to (49.5, 90.2)
- moved TP5 1870.3 mm to (57.1, 90.2)
- moved TP3 1844.7 mm to (96.6, 77.7), turned to 180 degrees
- moved CX1 1830.8 mm to (102.9, 81.3), turned to 90 degrees
- moved TP1 1830.8 mm to (104.1, 54.6)
- moved TP2 1830.8 mm to (104.1, 48.3)
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Connections:
- new net 485_5V: 5V_IN.1, 5V_OUT.1
- new net 485_A: U11.6
- new net 485_B: U11.7
- new net 485_RX: RX_IN.1, RX_OUT.1
- new net 485_TX: TX_IN.1, TX_OUT.1
- new net N$10: C21.1, L3.2, TP42.TP, U7.1
- new net N$11: F4.1, TP43.TP, U7.6
- new net N$12: C24.1, L4.2, TP47.TP, U8.1
- new net N$13: F5.1, TP48.TP, U8.6
- new net N$14: C27.1, L5.2, TP52.TP, U9.1
- new net N$21: F6.1, TP53.TP, U9.6
- new net N$24: C30.1, L6.2, TP57.TP, U10.1
- new net N$25: F7.1, TP58.TP, U10.6
- new net N$26: U11.2
- new net N$27: U11.3
- new net N$31: U11.4
- new net N$6: C6.1, L2.2, TP37.TP, U6.1
- new net N$9: F1.1, TP38.TP, U6.6
- net +24V: now also C10.1, C11.1, C13.+, C23.+, C26.+, C29.+, C32.+, C9.1, CX1.1, CX1.2, D1.C, L2.1, L3.1, L4.1, L5.1, L6.1; no longer TP23.TP
- net +3V3: now also U11.8; no longer TP19.TP, U2.7, U2.9
- net 24V_IN: no longer C10.1, C11.1, C9.1, CX1.1, CX1.2, D1.C
- net CH2+: now also F1.2
- net CH2-: now also C12.1, TP39.TP, U6.5
- net CH3+: now also F4.2
- net CH3-: now also C22.1, TP44.TP, U7.5
- net CH4+: now also F5.2
- net CH4-: now also C25.1, TP49.TP, U8.5
- net CH5+: now also F6.2
- net CH5-: now also C28.1, TP54.TP, U9.5
- net CH6+: now also F7.2
- net CH6-: now also C31.1, TP59.TP, U10.5
- net DIM2: now also TP35.TP, U6.2
- net DIM3: now also TP40.TP, U7.2
- net DIM4: now also TP45.TP, U8.2
- net DIM5: now also TP50.TP, U9.2
- net DIM6: now also TP55.TP, U10.2
- net GND1: now also GND_IN.1, GND_OUT.1, U11.5, _GND_IN.1, _GND_OUT.1; no longer I2C_GND_IN.1, I2C_GND_OUT.1, TP12.TP
- net GND2: now also C1.2, C12.2, C13.-, C2.2, C21.2, C22.2, C23.-, C24.2, C25.2, C26.-, C27.2, C28.2, C29.-, C30.2, C31.2, C32.-, C33.2, C6.2, C7.2, R12.1, TP36.TP, TP41.TP, TP46.TP, TP51.TP, TP56.TP, U$2.8, U10.4, U2.12, U2.13, U2.14, U6.4, U7.4, U8.4, U9.4; no longer R26.1, R28.1, R29.1, R30.1, TP20.TP, TP4.TP
- net I2C_3V3: now also 3V3_IN.1, 3V3_OUT.1; no longer I2C_3V3_IN.1, I2C_3V3_OUT.1, TP9.TP
- net I2C_SCL: now also SCL_IN.1, SCL_OUT.1; no longer I2C_SCL_IN.1, I2C_SCL_OUT.1, R6.1, TP11.TP
- net I2C_SDA: now also R6.1, SDA_IN.1, SDA_OUT.1; no longer I2C_SDA_IN.1, I2C_SDA_OUT.1, TP10.TP
- net N$1: no longer TP31.TP
- net N$15: now also R11.2, U2.5; no longer C7.2, R26.2
- net N$16: no longer TP34.TP
- net N$17: now also C33.1, R11.1; no longer C1.2, C2.2, R28.2
- net N$18: now also R12.2, U2.18; no longer R29.2, TP33.TP, U$2.8
- net N$19: now also U11.1; no longer R30.2, TP24.TP, U4.2
- net N$2: no longer TP32.TP
- net N$22: no longer TP27.TP
- net N$23: no longer TP25.TP
- net N$28: no longer TP28.TP
- net N$30: now also U4.2; no longer TP26.TP
- net N$4: no longer TP30.TP
- net N$7: no longer TP29.TP
- net N$8: no longer TP15.TP
- net SCL: no longer TP21.TP
- net SDA: no longer TP22.TP
Routing:
- net GND2: track 0.00 -> 131.4 mm, vias 0 -> 14
- net DIM6: track 0.00 -> 59.8 mm, vias 0 -> 1
- net DIM1: track 0.00 -> 58.9 mm, vias 0 -> 1
- net DIM2: track 0.00 -> 53.0 mm, vias 0 -> 2
- net DIM5: track 0.00 -> 50.1 mm, vias 0 -> 2
- net +3V3: track 0.00 -> 45.1 mm, vias 0 -> 18
- net DIM4: track 0.00 -> 30.0 mm, vias 0 -> 1
- net DIM3: track 0.00 -> 28.6 mm, vias 0 -> 1
- net N$30: track 0.00 -> 25.7 mm
- net GND1: track 0.00 -> 25.0 mm
- net N$14: track 0.00 -> 17.3 mm, vias 0 -> 1
- net N$6: track 0.00 -> 17.3 mm, vias 0 -> 1
- net N$3: track 0.00 -> 17.3 mm, vias 0 -> 1
- net N$12: track 0.00 -> 17.3 mm, vias 0 -> 1
- net N$10: track 0.00 -> 17.3 mm, vias 0 -> 1
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- added copper zone on layer 1, net +24V
- added copper zone on layer 1, net +3V3
- added copper zone on layer 16, net +3V3
- added copper zone on layer 1, net 24V_IN
- added copper zone on layer 16, net 485_5V
- added copper zone on layer 16, net 485_RX
- added copper zone on layer 16, net 485_TX
- added copper zone on layer 1, net CH1+
- added copper zone on layer 1, net CH1-
- added copper zone on layer 1, net CH2+
- added copper zone on layer 1, net CH2-
- added copper zone on layer 1, net CH3+
- added copper zone on layer 1, net CH3-
- added copper zone on layer 1, net CH4+
- added copper zone on layer 1, net CH4-
- added copper zone on layer 1, net CH5+
- added copper zone on layer 1, net CH5-
- added copper zone on layer 1, net CH6+
- added copper zone on layer 1, net CH6-
- added copper zone on layer 16, net CH6-
- added copper zone on layer 1, net GND
- added copper zone on layer 1, net GND2
- added copper zone on layer 16, net GND2
- added copper zone on layer 1, net N$10
- added copper zone on layer 1, net N$11
- added copper zone on layer 1, net N$12
- added copper zone on layer 1, net N$13
- added copper zone on layer 1, net N$14
- added copper zone on layer 1, net N$15
- added copper zone on layer 1, net N$17
- added copper zone on layer 1, net N$21
- added copper zone on layer 1, net N$24
- added copper zone on layer 1, net N$25
- added copper zone on layer 1, net N$3
- added copper zone on layer 1, net N$33
- added copper zone on layer 1, net N$5
- added copper zone on layer 1, net N$6
- added copper zone on layer 1, net N$9
Other:
- board size 100 x 80 mm -> 115.6 x 111.8 mm
